File: BatteryManagementUnit.kicad_pcb (KiCad board)
At the start: 2 copper layers, 3 parts, among them U2 AMC1301

Commit message: partial layout
Parts:
- added C201: 4.7nF, Capacitors_SMD:C_1206, F.Cu at (91.4, 152.4)
- added D201: PESD1CAN, TO_SOT_Packages_SMD:SOT-23_Handsoldering, F.Cu at (94.0, 121.9)
- added J201: RJ45, Connect:RJ45_8, F.Cu at (61.0, 141.0)
- added J202: RJ45, Connect:RJ45_8, F.Cu at (86.4, 141.0)
- added JP201: Terminate, electric_car_lib:JumperSingle, F.Cu at (63.5, 152.4)
- added JP202: Terminate, electric_car_lib:JumperSingle, F.Cu at (77.5, 158.8)
- added JP203: Filter, electric_car_lib:JumperSingle, F.Cu at (83.8, 152.4)
- added P1: HALL EFFECT, Pin_Headers:Pin_Header_Angled_1x04, F.Cu at (128.3, 138.4)
- added P101: HALL EFFECT, Pin_Headers:Pin_Header_Angled_1x04, F.Cu at (128.3, 125.7)
- added P102: CONN_01X02, Pin_Headers:Pin_Header_Angled_1x02, F.Cu at (114.3, 154.9)
- added P103: CONN_01X02, Pin_Headers:Pin_Header_Angled_1x02, F.Cu at (132.1, 163.8)
- added P104: CONT_H_mon, Connect:bornier2, F.Cu at (153.7, 39.4)
- added P105: CONT_L_mon, Connect:bornier2, F.Cu at (95.2, 21.6)
- added P106: CONT_H, Connect:bornier2, F.Cu at (36.8, 146.1)
- added P107: CONT_L, Connect:bornier2, F.Cu at (58.4, 124.5)
- added P2: CONN_01X02, Pin_Headers:Pin_Header_Angled_1x02, F.Cu at (130.8, 154.9)
- added P3: CONN_01X02, Pin_Headers:Pin_Header_Angled_1x02, F.Cu at (114.3, 163.8)
- added P4: CONT_H, Connect:bornier2, F.Cu at (101.6, 134.6)
- added P5: CONT_L, Connect:bornier2, F.Cu at (36.8, 135.9)
- added Q1: Q_NMOS_DGS, TO_SOT_Packages_SMD:TO-252-2Lead, F.Cu at (102.9, 127.0)
- added Q101: Q_NPN_BCE, TO_SOT_Packages_SMD:SOT-23_Handsoldering, F.Cu at (74.9, 22.9)
- added Q102: Q_NMOS_DGS, TO_SOT_Packages_SMD:TO-252-2Lead, F.Cu at (104.1, 148.6)
- added Q103: Q_NMOS_DGS, TO_SOT_Packages_SMD:TO-252-2Lead, F.Cu at (47.0, 125.7)
- added Q2: Q_NMOS_DGS, TO_SOT_Packages_SMD:TO-252-2Lead, F.Cu at (34.3, 125.7)
- added R101: R, Resistors_SMD:R_1210_HandSoldering, F.Cu at (108.0, 109.2)
- added R102: R, Resistors_SMD:R_1210_HandSoldering, F.Cu at (110.5, 115.6)
- added R201: 100, Resistors_SMD:R_1210_HandSoldering, F.Cu at (58.4, 118.1)
- added R202: 330, Resistors_SMD:R_1210_HandSoldering, F.Cu at (80.0, 114.3)
- added R203: 4.7K, Resistors_SMD:R_1210_HandSoldering, F.Cu at (76.2, 125.7)
- added R204: 60, Resistors_SMD:R_1210_HandSoldering, F.Cu at (73.7, 152.4)
- added R205: 60, Resistors_SMD:R_1210_HandSoldering, F.Cu at (69.8, 158.8)
- added U102: AMC1301, electric_car_lib:amc1301, F.Cu at (119.4, 109.2)
- added U201: TLP2361, electric_car_lib:soic-5, F.Cu at (68.6, 111.8)
- added U202: TLP2361, electric_car_lib:soic-5, F.Cu at (68.6, 120.7)
- added U203: MCP2551-I/SN, Power_Integrations:SO-8, F.Cu at (83.8, 121.9)
- moved U2 82.5 mm to (119.4, 101.6)
- moved R1 51.5 mm to (101.6, 113.0)
- moved R2 41.8 mm to (106.7, 104.1)
Connections:
- R1 pad 1: (no net) -> Net-(R1-Pad1)
- U2 pad 1: (no net) -> Net-(U2-Pad1)
- U2 pad 2: (no net) -> Net-(U2-Pad2)
- U2 pad 5: (no net) -> /Bat_Vn
- U2 pad 6: (no net) -> /Bat_Vp
- U2 pad 7: (no net) -> Net-(U2-Pad7)
- U2 pad 8: (no net) -> Net-(U2-Pad8)
Routing:
- net GNDREF: track 0.00 -> 112.5 mm, vias 0 -> 8
- net +12V: track 0.00 -> 98.8 mm, vias 0 -> 4
- net GNDA: track 0.00 -> 86.8 mm, vias 0 -> 2
- net /CANmodule/CAN_H: track 0.00 -> 79.9 mm, vias 0 -> 3
- net /CANmodule/CAN_L: track 0.00 -> 78.3 mm, vias 0 -> 2
- net Net-(P106-Pad1): track 0.00 -> 73.7 mm, vias 0 -> 4
- net /CNT_H: track 0.00 -> 32.6 mm, vias 0 -> 2
- net Net-(R1-Pad2): track 0.00 -> 22.1 mm
- net +5VA: track 0.00 -> 21.5 mm, vias 0 -> 2
- net /c_m_H_p: track 0.00 -> 17.8 mm
- net /c_m_H_n: track 0.00 -> 17.8 mm
- net /c_m_L_p: track 0.00 -> 16.5 mm
- net /c_m_L_n: track 0.00 -> 16.5 mm
- net Net-(JP203-Pad1): track 0.00 -> 15.1 mm
- net Net-(R202-Pad1): track 0.00 -> 14.9 mm
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
Commit message: completed schematic
Parts:
- removed P1: HALL EFFECT, Pin_Headers:Pin_Header_Angled_1x04
- removed P2, P3: CONN_01X02, Pin_Headers:Pin_Header_Angled_1x02
- removed P4: CONT_H, Connect:bornier2
- removed P5: CONT_L, Connect:bornier2
- removed Q1, Q2: Q_NMOS_DGS, TO_SOT_Packages_SMD:TO-252-2Lead
- removed R1, R2: R, Resistors_SMD:R_1210_HandSoldering
- removed U2: AMC1301, electric_car_lib:amc1301
- added J101: 0, Resistors_SMD:R_1210_HandSoldering, F.Cu at (243.5, 87.7)
- added P108: Battery, Connect:bornier2, F.Cu at (180.7, 128.5)
- added P109: PSU_ISO_3v, Pin_Headers:Pin_Header_Angled_1x04, F.Cu at (227.2, 39.5)
- added P110: PSU_ISO_5v, Pin_Headers:Pin_Header_Angled_1x04, F.Cu at (227.5, 66.7)
- added Q104: Q_NPN_BCE, TO_SOT_Packages_SMD:SOT-23_Handsoldering, F.Cu at (56.0, 50.1)
- added Q105: Q_NPN_BCE, TO_SOT_Packages_SMD:SOT-23_Handsoldering, F.Cu at (45.7, 46.4)
- added R103: 1k, Resistors_SMD:R_1210_HandSoldering, F.Cu at (28.7, 45.6)
- added R104: 1k, Resistors_SMD:R_1210_HandSoldering, F.Cu at (55.2, 39.9)
- added R105: 10k 2W, Resistors_ThroughHole:Resistor_Cement_KOA-BGR-3N, F.Cu at (53.5, 31.3)
- added R106: 120, Resistors_SMD:R_1210_HandSoldering, F.Cu at (142.2, 115.4)
- added R107: 120, Resistors_SMD:R_1210_HandSoldering, F.Cu at (39.8, 73.0)
- added R108: 1k, Resistors_SMD:R_1210_HandSoldering, F.Cu at (22.0, 35.0)
- added R109: 1k, Resistors_SMD:R_1210_HandSoldering, F.Cu at (31.2, 37.8)
- added R110: 10K 2W, Resistors_ThroughHole:Resistor_Cement_KOA-BGR-3N, F.Cu at (69.7, 52.1)
- added R111: 120, Resistors_SMD:R_1210_HandSoldering, F.Cu at (47.4, 66.2)
- added R112: 33, Resistors_SMD:R_1210_HandSoldering, F.Cu at (81.0, 99.0)
- added R113: 33, Resistors_SMD:R_1210_HandSoldering, F.Cu at (62.0, 109.5)
- added U103: Teensy_3.2, electric_car_lib:Teensy3.2_inv, F.Cu at (89.2, 138.8)
- added U104: TLP2361, electric_car_lib:soic-5, F.Cu at (37.7, 59.9)
- added U106: AP1117D33, TO_SOT_Packages_SMD:TO-263-3Lead, F.Cu at (213.7, 112.1)
- added U107: AP1117E50, TO_SOT_Packages_SMD:TO-263-3Lead, F.Cu at (221.3, 129.5)
- added U108: TLP2361, electric_car_lib:soic-5, F.Cu at (39.6, 35.8)
- P102: value CONN_01X02 -> cellsL
- P103: value CONN_01X02 -> cellsH
- moved P103 144.6 mm to (227.5, 55.2)
- moved P101 143.0 mm to (227.6, 22.9), turned to 0 degrees
- moved Q101 111.9 mm to (125.4, 122.7)
- moved P106 97.6 mm to (81.6, 59.3), turned to 90 degrees
- moved J201 95.0 mm to (155.6, 148.9)
- moved P107 91.0 mm to (91.9, 39.9), turned to 90 degrees
- moved P104 84.5 mm to (69.2, 38.7)
- moved P102 81.8 mm to (132.5, 75.2)
- moved JP201 72.2 mm to (133.4, 134.4)
- moved R201 71.5 mm to (119.3, 155.5)
- moved JP202 69.9 mm to (141.0, 129.6)
- moved JP203 63.2 mm to (144.5, 134.6)
- moved P105 57.8 mm to (59.1, 66.6)
- moved U201 54.7 mm to (110.8, 146.5), turned to 0 degrees
- moved R202 52.8 mm to (119.3, 149.5)
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Connections:
- net Net-(R102-Pad2) renamed /HV-
- P101 pad 1: /voltage5v -> +3V3
- P101 pad 2: /ground -> GND
- Q101 pad 2: Net-(Q101-Pad2) -> /HV+
- Q102 pad 2: /CNT_H -> Net-(Q102-Pad2)
- Q103 pad 2: /CNT_L -> Net-(Q103-Pad2)
- R101 pad 1: Net-(R101-Pad1) -> Net-(Q101-Pad3)
- U102 pad 1: Net-(U102-Pad1) -> /5v_Traction
- U102 pad 2: Net-(U102-Pad2) -> /GND_Traction
- U102 pad 7: Net-(U102-Pad7) -> GND
- U102 pad 8: Net-(U102-Pad8) -> +3V3
Routing:
- net /CANmodule/CAN_H: track 79.9 -> 0.00 mm, vias 3 -> 0
- net GNDREF: track 112.5 -> 33.2 mm, vias 8 -> 2
- net /CANmodule/CAN_TX: track 0.00 -> 79.1 mm, vias 0 -> 2
- net /CANmodule/CAN_L: track 78.3 -> 0.00 mm, vias 2 -> 0
- net Net-(P106-Pad1): track 73.7 -> 0.00 mm, vias 4 -> 0
- net +12V: track 98.8 -> 48.0 mm, vias 4 -> 0
- net /HV-: track 5.02 -> 53.6 mm
- net Net-(Q103-Pad2): track 0.00 -> 43.1 mm
- net /CANmodule/CAN_RX: track 0.00 -> 42.5 mm, vias 0 -> 4
- net /CNT_H: track 32.6 -> 62.9 mm
- net Net-(JP203-Pad1): track 15.1 -> 40.8 mm, vias 0 -> 2
- net GNDA: track 86.8 -> 64.4 mm, vias 2 -> 0
- net Net-(R1-Pad2): track 22.1 -> 0.00 mm
- net Net-(R203-Pad2): track 13.8 -> 34.4 mm, vias 0 -> 2
- net Net-(JP202-Pad2): track 14.1 -> 33.7 mm, vias 0 -> 2
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Other:
- board outline added: 135 x 0.1 mm

Commit message: changed footprints, corrected psu, grouped parts
Parts:
- added C101: C, Capacitors_SMD:C_1210_HandSoldering, F.Cu at (147.3, 68.6)
- added C102: C, Capacitors_SMD:C_1210_HandSoldering, F.Cu at (146.1, 55.9)
- added D101: D, Diodes_SMD:DO-214AB_Handsoldering, F.Cu at (206.4, 137.2)
- added D102: D, Diodes_SMD:DO-214AB_Handsoldering, F.Cu at (64.1, 128.9)
- added D103: D, Diodes_SMD:DO-214AB_Handsoldering, F.Cu at (89.5, 136.5)
- added J102: 0, Resistors_SMD:R_1210_HandSoldering, F.Cu at (139.1, 33.7)
- added R114: R, Resistors_SMD:R_1206_HandSoldering, F.Cu at (226.7, 148.6)
- added R115: 120, Resistors_SMD:R_1206_HandSoldering, F.Cu at (79.4, 36.2)
- added R116: 120, Resistors_SMD:R_1206_HandSoldering, F.Cu at (81.9, 45.1)
- added R117: 120, Resistors_SMD:R_1206_HandSoldering, F.Cu at (97.2, 62.2)
- added R118: 120, Resistors_SMD:R_1206_HandSoldering, F.Cu at (95.2, 49.5)
- added R119: 120, Resistors_SMD:R_1206_HandSoldering, F.Cu at (104.8, 131.4)
- added R120: 120, Resistors_SMD:R_1206_HandSoldering, F.Cu at (126.4, 135.3)
- added U101: FODM3052, electric_car_lib:MFP4L, F.Cu at (193.0, 134.6)
- added U105: FODM3052, electric_car_lib:MFP4L, F.Cu at (63.5, 109.2)
- added U109: FODM3052, electric_car_lib:MFP4L, F.Cu at (80.6, 112.4)
- added U110: TLP2361, electric_car_lib:soic-5, F.Cu at (107.3, 128.9)
- added U111: TLP2361, electric_car_lib:soic-5, F.Cu at (117.5, 129.5)
- C201: footprint Capacitors_SMD:C_1206 -> Capacitors_SMD:C_1210_HandSoldering
- P101, P109, P110: footprint Pin_Headers:Pin_Header_Angled_1x04 -> Pin_Headers:Pin_Header_Straight_1x04
- P102, P103: footprint Pin_Headers:Pin_Header_Angled_1x02 -> Pin_Headers:Pin_Header_Straight_1x02
- Q101, Q104, Q105: footprint TO_SOT_Packages_SMD:SOT-23_Handsoldering -> TO_SOT_Packages_SMD:TO-252-2Lead
- Q102, Q103: value Q_NMOS_DGS -> Q_NMOS_GDS
- R101, R102, R103, R104, R106, R107, R108, R109, R111, R112, R113, R201, R202, R203, R204, R205: footprint Resistors_SMD:R_1210_HandSoldering -> Resistors_SMD:R_1206_HandSoldering
- U103: footprint electric_car_lib:Teensy3.2_inv -> electric_car_lib:Teensy3.2
- U106, U107: footprint TO_SOT_Packages_SMD:TO-263-3Lead -> TO_SOT_Packages_SMD:SOT-223
- moved R202 162.6 mm to (280.0, 125.1)
- moved P103 160.2 mm to (67.9, 40.0)
- moved R203 156.5 mm to (247.0, 52.1)
- moved U203 155.2 mm to (237.5, 48.3)
- moved U201 153.5 mm to (262.3, 121.3)
- moved J202 145.0 mm to (219.1, 32.4), turned to 180 degrees
- moved J201 143.5 mm to (239.4, 32.4), turned to 180 degrees
- moved R204 142.8 mm to (245.7, 68.6)
- moved R205 141.0 mm to (233.0, 64.8)
- moved C201 139.3 mm to (254.0, 56.5)
- moved U202 134.6 mm to (237.5, 122.6)
- moved P107 130.3 mm to (123.2, 166.4), turned to 0 degrees
- moved JP201 126.5 mm to (233.0, 56.5)
- moved P104 124.5 mm to (57.1, 162.6)
- moved JP203 123.8 mm to (242.6, 59.1)
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Connections:
- net /HV+ renamed Net-(D101-Pad1)
- net /HV- renamed Net-(P108-Pad2)
- J101 pad 1: GNDA -> Net-(J101-Pad1)
- J101 pad 2: GND -> +5VA
- P102 pad 1: /c_m_L_n -> Net-(P102-Pad1)
- P102 pad 2: /c_m_L_p -> Net-(P102-Pad2)
- P103 pad 1: /c_m_H_n -> Net-(P103-Pad1)
- P103 pad 2: /c_m_H_p -> Net-(P103-Pad2)
- P109 pad 1: +12V -> GNDA
- P109 pad 2: GNDA -> +12V
- P110 pad 1: +12V -> GNDA
- P110 pad 2: GND -> +12V
- Q102 pad 1: Net-(P106-Pad1) -> Net-(Q102-Pad1)
- Q102 pad 2: Net-(Q102-Pad2) -> Net-(P106-Pad1)
- Q102 pad 3: GNDREF -> GNDA
- Q103 pad 1: Net-(P107-Pad1) -> Net-(Q103-Pad1)
- Q103 pad 2: Net-(Q103-Pad2) -> Net-(P107-Pad1)
- Q103 pad 3: GNDREF -> GNDA
- R111 pad 1: /PrechargeL -> Net-(R111-Pad1)
- R111 pad 2: Net-(R111-Pad2) -> /PrechargeL
- R112 pad 1: /CNT_H -> Net-(R112-Pad1)
- R112 pad 2: Net-(Q102-Pad2) -> Net-(Q102-Pad1)
- R113 pad 1: /CNT_L -> Net-(R113-Pad1)
- R113 pad 2: Net-(Q103-Pad2) -> Net-(Q103-Pad1)
- U102 pad 3: Net-(R101-Pad2) -> Net-(R114-Pad1)
- U103 pad 1: Net-(U103-Pad1) -> GND
- U103 pad 13: Net-(R111-Pad2) -> /PrechargeL
- U103 pad 26: Net-(U103-Pad26) -> +3V3
- U106 pad 3: +5VA -> Net-(J101-Pad1)
Routing:
- net /CANmodule/CAN_TX: track 79.1 -> 0.00 mm, vias 2 -> 0
- net GNDA: track 64.4 -> 0.00 mm
- net /CNT_H: track 62.9 -> 0.00 mm, vias 2 -> 0
- net Net-(P108-Pad2): track 53.6 -> 0.00 mm
- net +12V: track 48.0 -> 0.00 mm
- net Net-(Q103-Pad2): track 43.1 -> 0.00 mm
- net /CANmodule/CAN_RX: track 42.5 -> 0.00 mm, vias 4 -> 0
- net Net-(JP203-Pad1): track 40.8 -> 0.00 mm, vias 2 -> 0
- net Net-(R203-Pad2): track 34.4 -> 0.00 mm, vias 2 -> 0
- net Net-(JP202-Pad2): track 33.7 -> 0.00 mm, vias 2 -> 0
- net GNDREF: track 33.2 -> 0.00 mm, vias 2 -> 0
- net +5VA: track 23.2 -> 0.00 mm, vias 6 -> 0
- net Net-(R202-Pad1): track 22.6 -> 0.00 mm, vias 2 -> 0
- net Net-(R101-Pad2): track 18.2 -> 0.00 mm
- net +3V3: track 14.4 -> 0.00 mm
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Other:
- board size 135 x 0.1 mm -> 0.1 x 0.1 mm
