File: CANmodule.sch (KiCad schematic (older format))
At the start: 15 parts, among them J201 RJ45, J202 RJ45, U201 TLP2361, U202 TLP2361, U203 MCP2551-I/SN

Commit message: changed footprints, corrected psu, grouped parts
Parts:
- C201: footprint Capacitors_SMD:C_1206 -> Capacitors_SMD:C_1210_HandSoldering
- R201, R202, R203, R204, R205: footprint Resistors_SMD:R_1210_HandSoldering -> Resistors_SMD:R_1206_HandSoldering
Changed lines of the file:
@@
 F 0 "R203" V 6930 2000 50  0000 C CNN
 F 1 "4.7K" V 6850 2000 50  0000 C CNN
-F 2 "Resistors_SMD:R_1210_HandSoldering" V 6780 2000 50  0001 C CNN
+F 2 "Resistors_SMD:R_1206_HandSoldering" V 6780 2000 50  0001 C CNN
 F 3 "" H 6850 2000 50  0000 C CNN
 	1    6850 2000
@@
 F 0 "C201" H 8725 2600 50  0000 L CNN
 F 1 "4.7nF" H 8725 2400 50  0000 L CNN
-F 2 "Capacitors_SMD:C_1206" H 8738 2350 50  0001 C CNN
+F 2 "Capacitors_SMD:C_1210_HandSoldering" H 8738 2350 50  0001 C CNN
 F 3 "" H 8700 2500 50  0000 C CNN
 	1    8700 2500
@@
 F 0 "R204" V 8030 2350 50  0000 C CNN
 F 1 "60" V 7950 2350 50  0000 C CNN
-F 2 "Resistors_SMD:R_1210_HandSoldering" V 7880 2350 50  0001 C CNN
+F 2 "Resistors_SMD:R_1206_HandSoldering" V 7880 2350 50  0001 C CNN
 F 3 "" H 7950 2350 50  0000 C CNN
 	1    7950 2350
@@
 F 0 "R205" V 8230 2350 50  0000 C CNN
 F 1 "60" V 8150 2350 50  0000 C CNN
-F 2 "Resistors_SMD:R_1210_HandSoldering" V 8080 2350 50  0001 C CNN
+F 2 "Resistors_SMD:R_1206_HandSoldering" V 8080 2350 50  0001 C CNN
 F 3 "" H 8150 2350 50  0000 C CNN
 	1    8150 2350
@@
 F 0 "R202" V 6380 1450 50  0000 C CNN
 F 1 "330" V 6300 1450 50  0000 C CNN
-F 2 "Resistors_SMD:R_1210_HandSoldering" V 6230 1450 50  0001 C CNN
+F 2 "Resistors_SMD:R_1206_HandSoldering" V 6230 1450 50  0001 C CNN
 F 3 "" H 6300 1450 50  0000 C CNN
 	1    6300 1450
@@
 F 0 "R201" V 4880 2050 50  0000 C CNN
 F 1 "100" V 4800 2050 50  0000 C CNN
-F 2 "Resistors_SMD:R_1210_HandSoldering" V 4730 2050 50  0001 C CNN
+F 2 "Resistors_SMD:R_1206_HandSoldering" V 4730 2050 50  0001 C CNN
 F 3 "" H 4800 2050 50  0000 C CNN
 	1    4800 2050
@@
 $EndComp
 $Comp
-L GND #PWR028
+L GND #PWR036
 U 1 1 57FCAEF7
 P 5150 1700
-F 0 "#PWR028" H 5150 1450 50  0001 C CNN
+F 0 "#PWR036" H 5150 1450 50  0001 C CNN
 F 1 "GND" H 5150 1550 50  0000 C CNN
 F 2 "" H 5150 1700 50  0000 C CNN
@@
 CAN_L
 $Comp
-L +5VA #PWR029
+L +5VA #PWR037
 U 1 1 582A8343
 P 6000 1400
-F 0 "#PWR029" H 6000 1250 50  0001 C CNN
+F 0 "#PWR037" H 6000 1250 50  0001 C CNN
 F 1 "+5VA" H 6000 1540 50  0000 C CNN
 F 2 "" H 6000 1400 50  0000 C CNN
@@
 $EndComp
 $Comp
-L +5VA #PWR030
+L +5VA #PWR038
 U 1 1 582A84BF
 P 7200 1000
-F 0 "#PWR030" H 7200 850 50  0001 C CNN
+F 0 "#PWR038" H 7200 850 50  0001 C CNN
 F 1 "+5VA" H 7200 1140 50  0000 C CNN
 F 2 "" H 7200 1000 50  0000 C CNN
@@
 $EndComp
 $Comp
-L GNDA #PWR031
+L GNDA #PWR039
 U 1 1 582A8520
 P 6000 2300
-F 0 "#PWR031" H 6000 2050 50  0001 C CNN
+F 0 "#PWR039" H 6000 2050 50  0001 C CNN
 F 1 "GNDA" H 6000 2150 50  0000 C CNN
 F 2 "" H 6000 2300 50  0000 C CNN
@@
 $EndComp
 $Comp
-L GNDA #PWR032
+L GNDA #PWR040
 U 1 1 582A8593
 P 7200 2100
-F 0 "#PWR032" H 7200 1850 50  0001 C CNN
+F 0 "#PWR040" H 7200 1850 50  0001 C CNN
 F 1 "GNDA" H 7200 1950 50  0000 C CNN
 F 2 "" H 7200 2100 50  0000 C CNN
@@
 $EndComp
 $Comp
-L GNDA #PWR033
+L GNDA #PWR041
 U 1 1 582A864A
 P 9450 1650
-F 0 "#PWR033" H 9450 1400 50  0001 C CNN
+F 0 "#PWR041" H 9450 1400 50  0001 C CNN
 F 1 "GNDA" H 9450 1500 50  0000 C CNN
 F 2 "" H 9450 1650 50  0000 C CNN
@@
 $EndComp
 $Comp
-L GNDA #PWR034
+L GNDA #PWR042
 U 1 1 582A86D1
 P 9050 2500
-F 0 "#PWR034" H 9050 2250 50  0001 C CNN
+F 0 "#PWR042" H 9050 2250 50  0001 C CNN
 F 1 "GNDA" H 9050 2350 50  0000 C CNN
 F 2 "" H 9050 2500 50  0000 C CNN
@@
 $EndComp
 $Comp
-L +3V3 #PWR035
+L +3V3 #PWR043
 U 1 1 582A8930
 P 5000 1400
-F 0 "#PWR035" H 5000 1250 50  0001 C CNN
+F 0 "#PWR043" H 5000 1250 50  0001 C CNN
 F 1 "+3V3" H 5000 1540 50  0000 C CNN
 F 2 "" H 5000 1400 50  0000 C CNN
@@
 $EndComp
 $Comp
-L +12V #PWR036
+L +12V #PWR044
 U 1 1 582DA73C
 P 8200 5000
-F 0 "#PWR036" H 8200 4850 50  0001 C CNN
+F 0 "#PWR044" H 8200 4850 50  0001 C CNN
 F 1 "+12V" H 8200 5140 50  0000 C CNN
 F 2 "" H 8200 5000 50  0000 C CNN
@@
 $EndComp
 $Comp
-L GNDA #PWR037
+L GNDA #PWR045
 U 1 1 582DA7E4
 P 8400 5000
-F 0 "#PWR037" H 8400 4750 50  0001 C CNN
+F 0 "#PWR045" H 8400 4750 50  0001 C CNN
 F 1 "GNDA" H 8400 4850 50  0000 C CNN
 F 2 "" H 8400 5000 50  0000 C CNN
@@
 $EndComp
 $Comp
-L +12V #PWR038
+L +12V #PWR046
 U 1 1 582DC5D0
 P 7100 5000
-F 0 "#PWR038" H 7100 4850 50  0001 C CNN
+F 0 "#PWR046" H 7100 4850 50  0001 C CNN
 F 1 "+12V" H 7100 5140 50  0000 C CNN
 F 2 "" H 7100 5000 50  0000 C CNN
@@
 $EndComp
 $Comp
-L GNDA #PWR039
+L GNDA #PWR047
 U 1 1 582DC5D6
 P 7300 5000
-F 0 "#PWR039" H 7300 4750 50  0001 C CNN
+F 0 "#PWR047" H 7300 4750 50  0001 C CNN
 F 1 "GNDA" H 7300 4850 50  0000 C CNN
 F 2 "" H 7300 5000 50  0000 C CNN
